Commit message: new demo world

File: pycram/resources/worlds/apartment_without_walls.urdf (robot description, URDF)
Before this commit: robot apartment, 106 links, 105 joints
Links:
- added link table_area_main, mass 1; collision mesh filename=package://iai_kitchen/meshes/misc/big_table_1.obj; visual mesh filename=package://iai_kitchen/meshes/misc/big_table_1.dae
Joints:
- added joint table_area_main_joint: type fixed, parent apartment_root, child table_area_main, origin xyz=5 4 0 rpy=0 0 1.57
