Commit message: more refactor

File: pycram/resources/worlds/apartment_without_walls.urdf (robot description, URDF)
Before this commit: robot apartment, 107 links, 106 joints
Links:
- removed link table_area_main
Joints:
- removed joint table_area_main_joint

File: pycram/resources/worlds/kitchen.urdf (robot description, URDF)
Before this commit: robot iai_oven_area, 84 links, 83 joints
Joints:
- joint sink_area_dish_washer_door_joint: limit lower=0 upper=1.57079632679 effort=300 velocity=10 -> lower=0 upper=0 effort=300 velocity=10
- joint sink_area_dish_washer_main_joint: axis (none) -> 1 0 0; limit (none) -> lower=0 upper=0 effort=300 velocity=10; type fixed -> revolute
