Commit message: world

File: pycram/resources/worlds/kitchen.urdf (robot description, URDF)
Before this commit: robot iai_oven_area, 84 links, 83 joints
Joints:
- joint sink_area_dish_washer_door_joint: limit lower=0 upper=0 effort=300 velocity=10 -> lower=0 upper=1.57079632679 effort=300 velocity=10
- joint sink_area_dish_washer_main_joint: axis 1 0 0 -> (none); limit lower=0 upper=0 effort=300 velocity=10 -> (none); type revolute -> fixed
